Commit message: kistar_son: thumb_2 joint axis -Y for URDF/MuJoCo consistency
Made-with: Cursor

File: robots/hands/kistar_son/kistar_son_left_mockup.urdf (robot description, URDF)
Before this commit: robot KISTAR_SON_LEFT, 62 links, 60 joints
Joints:
- joint left_hand_thumb_2_joint: axis 0 1 0 -> 0 -1 0

File: robots/hands/kistar_son/kistar_son_right_mockup.urdf (robot description, URDF)
Before this commit: robot KISTAR_SON_RIGHT, 62 links, 60 joints
Joints:
- joint right_hand_thumb_2_joint: axis 0 1 0 -> 0 -1 0
