Commit message: kistar_son: add palm back_2 link (URDF + MJCF, both hands)
- Add left/right_hand_base_back_2_link mesh, fixed joint, and MJCF geoms
- Update author affiliation header to PRIME Lab in URDFs
- Unify position actuator gains (kp=30 kv=0.7 forcerange=-100 100) in right URDF
- Ignore 20260522_KISTAR_SON_URDF_BI/ working folder

Co-authored-by: Cursor <cursoragent@cursor.com>

File: robots/hands/kistar_son/kistar_son_left_mockup.urdf (robot description, URDF)
Before this commit: robot KISTAR_SON_LEFT, 62 links, 60 joints
Links:
- added link left_hand_base_back_2_link, mass 0.; collision mesh filename=01_kistar_son_STL/left_hand_base_back_2_link.STL; visual mesh filename=01_kistar_son_STL/left_hand_base_back_2_link.STL
Joints:
- added joint left_hand_base_back_2_joint: type fixed, parent left_hand_base_link, child left_hand_base_back_2_link, origin xyz=0. 0. 0. rpy=0. 0. 0.

File: robots/hands/kistar_son/kistar_son_right_mockup.urdf (robot description, URDF)
Before this commit: robot KISTAR_SON_RIGHT, 62 links, 60 joints
Links:
- added link right_hand_base_back_2_link, mass 0.; collision mesh filename=01_kistar_son_STL/right_hand_base_back_2_link.STL; visual mesh filename=01_kistar_son_STL/right_hand_base_back_2_link.STL
Joints:
- added joint right_hand_base_back_2_joint: type fixed, parent right_hand_base_link, child right_hand_base_back_2_link, origin xyz=0. 0. 0. rpy=0. 0. 0.

Commit message: kistar_son: replace palm back_2 with front_2 link (URDF + MJCF, both hands)
- Add left/right_hand_base_front_2_link mesh, fixed joint, MJCF geoms
- Remove obsolete left/right_hand_base_back_2_link (mesh + URDF link + MJCF geom)
- Fix typo: empty kp="" in right URDF default position
- Sync robots/hands/kistar_son with 20260522 BI source

Co-authored-by: Cursor <cursoragent@cursor.com>

File: robots/hands/kistar_son/kistar_son_left_mockup.urdf (robot description, URDF)
Before this commit: robot KISTAR_SON_LEFT, 63 links, 61 joints
Links:
- removed link left_hand_base_back_2_link
- added link left_hand_base_front_2_link, mass 0.; collision mesh filename=01_kistar_son_STL/left_hand_base_front_2_link.STL; visual mesh filename=01_kistar_son_STL/left_hand_base_front_2_link.STL
Joints:
- removed joint left_hand_base_back_2_joint
- added joint left_hand_base_front_2_joint: type fixed, parent left_hand_base_link, child left_hand_base_front_2_link, origin xyz=0. 0. 0. rpy=0. 0. 0.

File: robots/hands/kistar_son/kistar_son_right_mockup.urdf (robot description, URDF)
Before this commit: robot KISTAR_SON_RIGHT, 63 links, 61 joints
Links:
- removed link right_hand_base_back_2_link
- added link right_hand_base_front_2_link, mass 0.; collision mesh filename=01_kistar_son_STL/right_hand_base_front_2_link.STL; visual mesh filename=01_kistar_son_STL/right_hand_base_front_2_link.STL
Joints:
- removed joint right_hand_base_back_2_joint
- added joint right_hand_base_front_2_joint: type fixed, parent right_hand_base_link, child right_hand_base_front_2_link, origin xyz=0. 0. 0. rpy=0. 0. 0.
